Commit message: Make the capstone fly, and score it
The reference solution now runs end to end against Gazebo ground truth and is
scored: 80/85 at tier 0, 68 at tier 1, 67 at tier 2. The first honest score was
13.3, and getting from there to here took six defects that were invisible from
reading the code and obvious from one measurement each. Every one of them is
written down next to the thing it broke, because each is also something the
course now teaches.

  * The detector ran at imgsz=640, where a 64 px target letterboxes down to
    32 px and YOLO finds no vehicle at all -- it reports an aeroplane at 0.73.
    960 finds the truck at 0.58 for 42 ms. The build now fails if the detector
    cannot find a vehicle in a frame taken from the air at the course geometry,
    not merely in a stock sample image.
  * Detection confidence collapses toward nadir: 0.51 at 40 degrees down, 0.27
    at 50, nothing past 60, because COCO contains almost no vehicles
    photographed from above. The detector, not the error model, chooses the
    flight geometry -- hence 12 m up and 18 m back.
  * The gimbal pointer's yaw sign was a guess and was backwards, so it drove the
    target out of frame. Measured and written down.
  * A pointer that only reacts to pixels never looks back, so one dropped frame
    lost the target for good. It now coasts on the filter's prediction,
    projected into the optical frame, feeding the same PID.
  * The velocity field of PositionTarget is a feedforward, not a control law.
    Sending Kp*e there doubles the gain against PX4's own MPC_XY_P: the aircraft
    ran 5 m past a stationary target and lost it.
  * "Hold overhead" is the wrong fallback for a stopped target. It is a nadir
    view, and detections go to zero while hovering over a truck in plain sight.

Two things were the simulation lying rather than the code being wrong. The
target spawned facing the aircraft and drove straight over it before takeoff,
shoving it 13 m and making tiers 2 and 3 score as if the follower had failed.
And the vendored pickup mesh has its length along its own +Y in inches, so the
truck drove sideways with its heading permanently 90 degrees from its velocity.

EKF2's yaw sits 5-6 degrees off truth in this simulator. That was chased until
it reproduced with stock PX4, the stock x500 and the stock world, so it is not
ours and cannot be tuned away from here. It is the largest term in the
geolocation error budget, and it is wired into the course rather than hidden:
the scoring thresholds allow for it and the error budget names attitude as the
dominant term, which is also true on the real aircraft.

Also in this change:

  * Ground truth for scoring, via one OdometryPublisher per scored model. This
    sidesteps the Pose_V link-name problem that blocked it, rather than solving
    it.
  * scoring_node.py and `course score`: the rubric, computed from ground truth.
  * Lab skeletons and reference solutions for labs 3, 4, 5 and the capstone,
    with `course new` and `course solution`. Skeletons are GENERATED from the
    solutions, so they cannot drift into something that can no longer become the
    answer they are graded against.
  * The frozen interface contract in exercises/INTERFACES.md.
  * QGroundControl v4.4.4 in the image, extracted rather than run.
  * A browser desktop fallback: `course desktop`, so no student is blocked by
    their laptop's graphics stack.
  * `course log`, because PX4 writes logs where a student cannot reach them, and
    `course rviz` with a canned layout.
  * Two SITL-only airframe defaults, COM_RC_IN_MODE and NAV_DLL_ACT, without
    which PX4 refuses to arm and says only "Resolve system health failures
    first".
  * Student-facing documentation: pre-work, troubleshooting by error message,
    hardware checklist, field procedure, syllabus.

Co-Authored-By: Claude Opus 5 (1M context) <noreply@anthropic.com>

File: ros2_ws/src/drone_course_sim/urdf/x500_course_gimbal.urdf.xacro (robot description, xacro)
@@ -15,4 +15,11 @@
   <xacro:property name="pi2" value="1.5707963267948966"/>
   <!-- Gimbal rotation centre relative to base_link. -->
+  <!-- Measured from a running simulation, not derived on paper: read the
+       link poses out of /world/course_world/pose/info and subtract base_link's.
+       The payload sits forward of and just below the airframe centre so the
+       camera does not look into a landing leg. Both numbers must track
+       models/x500_course_gimbal/model.sdf; a build-time check in the Dockerfile
+       fails if they drift apart. -->
+  <xacro:property name="mount_x" value="0.0"/>
   <xacro:property name="mount_z" value="0.02"/>
   <link name="base_link"/>
@@ -28,5 +35,5 @@
     <parent link="base_link"/>
     <child link="cgo3_mount_link"/>
-    <origin xyz="0 0 ${mount_z}" rpy="0 0 ${pi2*2}"/>
+    <origin xyz="${mount_x} 0 ${mount_z}" rpy="0 0 ${pi2*2}"/>
   </joint>
   <joint name="cgo3_vertical_arm_joint" type="revolute">   <!-- yaw -->

Commit message: Draw the aircraft in RViz, and pivot the gimbal frames where Gazebo does
The URDF had the three gimbal joints at zero translation, pivoting at the
mount. Gazebo pivots them about the SDF joint poses, 0.16 m lower at the
camera, so camera_optical_frame sat 16 cm above the lens and camera_link
was 0.10 m off at 35 deg pitch. course verify could not see it: it checks
at zero joint angles, the one pose where every link origin coincides.

Each link now sits at its joint's pivot and the optical frame at the
sensor. Names, axes, limits, rotations and the mount offset are
unchanged. TF matches Gazebo link poses to 1.4 mm / 0.5 deg across four
gimbal poses; six A/B capstone runs show no score effect.

Also:
- URDF visuals from the Gazebo meshes, installed into the package share
  from models/ by CMake (COURSE_MODELS_DIR), not copied in git
- RobotModel display in course.rviz
- make_media.sh frames: the Day 3 "frames on the aircraft" screenshot,
  with frame_axes.py drawing the axes from /tf (the TF display draws
  white names and ignored its frame filter)
- spike notes 41-44, PROGRESS entry, two open issues

Co-Authored-By: Claude Opus 5.5 <noreply@anthropic.com>

File: ros2_ws/src/drone_course_sim/urdf/x500_course_gimbal.urdf.xacro (robot description, xacro)
@@ -2,9 +2,17 @@
 <!--
   TF tree for the course aircraft.
-  The link origins are NOT guessed from the SDF: they were read out of a running
-  simulation. In the assembled model every gimbal link origin coincides at the
-  gimbal's rotation centre, which sits 0.02 m above base_link (base_link is at
-  z = 0.24 in the model frame, the gimbal is merged at z = 0.26). That is why
-  the three revolute joints below have zero translation.
+  Every number here was checked against a running simulation, not only read
+  off the SDF. The gimbal model frame sits 0.02 m above base_link (base_link is
+  at z = 0.24 in the model frame, the gimbal is merged at z = 0.26), and at
+  zero joint angles every gimbal link origin coincides with it.
+  That point is NOT where the gimbal rotates. Each SDF joint pivots about its
+  own point (the joint <pose>, in the child link), and the pitch pivot is
+  0.16 m lower, at the camera. An earlier version of this file put all three
+  revolute joints at zero translation, i.e. pivoting at the mount: rotations
+  right, positions wrong. camera_optical_frame sat 16 cm above the lens, and
+  at 35 deg of pitch Gazebo's camera_link was 0.10 m from where TF said. So
+  each link frame below is placed at its joint's pivot instead. Measured, at
+  34.6 deg pitch: a rotation about the SDF pivot predicts camera_link at
+  (0.0993, 0, 0.0147) from base_link, and Gazebo reports (0.0993, 0, 0.0147).
   Joint angles come from /joint_states. In simulation those are published by the
   model's JointStatePublisher; on the real aircraft the SIYI driver's attitude
@@ -14,5 +22,5 @@
 <robot xmlns:xacro="http://www.ros.org/wiki/xacro" name="x500_course_gimbal">
   <xacro:property name="pi2" value="1.5707963267948966"/>
-  <!-- Gimbal rotation centre relative to base_link. -->
+  <!-- Gimbal model frame relative to base_link. -->
   <!-- Measured from a running simulation, not derived on paper: read the
        link poses out of /world/course_world/pose/info and subtract base_link's.
@@ -23,9 +31,100 @@
   <xacro:property name="mount_x" value="0.0"/>
   <xacro:property name="mount_z" value="0.02"/>
-  <link name="base_link"/>
-  <link name="cgo3_mount_link"/>
-  <link name="cgo3_vertical_arm_link"/>
-  <link name="cgo3_horizontal_arm_link"/>
-  <link name="camera_link"/>
+  <!-- Joint pivots in the gimbal model frame, copied from the joint <pose>s
+       in models/course_gimbal/model.sdf (at zero angles every child link frame
+       is the model frame, so these need no conversion). The model frame is
+       yawed 180 deg from base_link: -x here is aircraft FORWARD. -->
+  <xacro:property name="yaw_px" value="-0.02552"/>                 <!-- cgo3_vertical_arm_joint -->
+  <xacro:property name="roll_pz" value="-0.1619"/>                 <!-- cgo3_horizontal_arm_joint -->
+  <xacro:property name="pitch_px" value="-0.0412"/>                <!-- cgo3_camera_joint -->
+  <xacro:property name="pitch_pz" value="-0.162"/>
+  <!-- The camera sensor, in the same frame: <sensor name="camera"> <pose>.
+       It sits 3.3 cm in front of the pitch pivot. -->
+  <xacro:property name="lens_px" value="-0.074"/>
+  <!--
+    Visuals, so RViz draws the aircraft under its frames. They are for looking
+    at only: nothing reads them, and they change no transform.
+    The meshes are the ones Gazebo renders, installed into this package's share
+    by CMakeLists.txt from models/: one copy in git, two consumers. Every
+    pose is copied from the SDF:
+      base_link  the SDF's base_link has the same frame as this one, so the
+                 body and motor-base poses are used as they are. The rotors are
+                 separate spinning links in the SDF; here they are fixed to
+                 base_link at (rotor link pose + rotor visual pose), which is
+                 a sum because none of those poses carries a rotation.
+      gimbal     every gimbal link in models/course_gimbal has an identity
+                 pose (all four coincide with the gimbal model frame), and each
+                 mesh is at the identity in its SDF link. The URDF links sit at
+                 their pivots instead, so each mesh is offset by minus its
+                 link's pivot, and then moves with the link exactly as
+                 Gazebo moves it.
+    If a mesh ever looks wrong in RViz, check it against the running
+    simulation before touching anything: the joints are the measured TF tree.
+  -->
+  <xacro:property name="mesh_x500" value="package://drone_course_sim/meshes/course_x500_base"/>
+  <xacro:property name="mesh_gimbal" value="package://drone_course_sim/meshes/course_gimbal"/>
+  <xacro:property name="prop_scale" value="0.8461538461538461"/>
+  <!-- Every visual names a material, the DAEs included (they keep their own
+       textures regardless). rviz2 looks only at a link's FIRST visual: if that
+       one has no material, every untextured mesh on the link is drawn in
+       RVIZ/ShadedRed, which is how the props came out red. -->
+  <material name="airframe"><color rgba="0.2 0.2 0.2 1"/></material>
+  <material name="prop_grey"><color rgba="0.25 0.25 0.25 1"/></material>
+  <material name="gimbal_grey"><color rgba="0.175 0.175 0.175 1"/></material>
+  <xacro:macro name="motor_and_prop" params="x y prop">
+    <visual>
+      <origin xyz="${x} ${y} 0.032" rpy="0 0 -0.45"/>
+      <geometry><mesh filename="${mesh_x500}/5010Base.dae"/></geometry>
+      <material name="airframe"/>
+    </visual>
+    <!-- rotor link at (x, y, 0.06); bell at -0.032 in it -->
+    <visual>
+      <origin xyz="${x} ${y} ${0.06 - 0.032}" rpy="0 0 0"/>
+      <geometry><mesh filename="${mesh_x500}/5010Bell.dae"/></geometry>
+      <material name="airframe"/>
+    </visual>
+    <!-- prop visual at (-0.022, -0.14638..., -0.016) in the rotor link: the
+         mesh origin is not at its hub -->
+    <visual>
+      <origin xyz="${x - 0.022} ${y - 0.14638461538461536} ${0.06 - 0.016}" rpy="0 0 0"/>
+      <geometry>
+        <mesh filename="${mesh_x500}/${prop}" scale="${prop_scale} ${prop_scale} ${prop_scale}"/>
+      </geometry>
+      <material name="prop_grey"/>
+    </visual>
+  </xacro:macro>
+  <link name="base_link">
+    <visual>
+      <origin xyz="0 0 0.025" rpy="0 0 ${pi2*2}"/>
+      <geometry><mesh filename="${mesh_x500}/NXP-HGD-CF.dae"/></geometry>
+      <material name="airframe"/>
+    </visual>
+    <!-- rotor_0..3 of the SDF, same numbering -->
+    <xacro:motor_and_prop x="0.174" y="-0.174" prop="1345_prop_ccw.stl"/>
+    <xacro:motor_and_prop x="-0.174" y="0.174" prop="1345_prop_ccw.stl"/>
+    <xacro:motor_and_prop x="0.174" y="0.174" prop="1345_prop_cw.stl"/>
+    <xacro:motor_and_prop x="-0.174" y="-0.174" prop="1345_prop_cw.stl"/>
+  </link>
+  <!-- px pz: the link's pivot in the gimbal model frame; the mesh is drawn
+       at minus that, which is where the SDF has it. -->
+  <xacro:macro name="gimbal_link" params="name mesh px pz">
+    <link name="${name}">
+      <visual>
+        <origin xyz="${-px} 0 ${-pz}" rpy="0 0 0"/>
+        <geometry>
+          <mesh filename="${mesh_gimbal}/${mesh}" scale="0.001 0.001 0.001"/>
+        </geometry>
+        <material name="gimbal_grey"/>
+      </visual>
+    </link>
+  </xacro:macro>
+  <xacro:gimbal_link name="cgo3_mount_link" mesh="cgo3_mount_remeshed_v1.stl"
+                     px="0" pz="0"/>
+  <xacro:gimbal_link name="cgo3_vertical_arm_link" mesh="cgo3_vertical_arm_remeshed_v1.stl"
+                     px="${yaw_px}" pz="0"/>
+  <xacro:gimbal_link name="cgo3_horizontal_arm_link" mesh="cgo3_horizontal_arm_remeshed_v1.stl"
+                     px="0" pz="${roll_pz}"/>
+  <xacro:gimbal_link name="camera_link" mesh="cgo3_camera_remeshed_v1.stl"
+                     px="${pitch_px}" pz="${pitch_pz}"/>
   <link name="camera_optical_frame"/>
   <!-- The mount carries a 180 deg yaw, exactly as the model does. It is kept
@@ -40,5 +139,5 @@
     <parent link="cgo3_mount_link"/>
     <child link="cgo3_vertical_arm_link"/>
-    <origin xyz="0 0 0" rpy="0 0 0"/>
+    <origin xyz="${yaw_px} 0 0" rpy="0 0 0"/>
     <axis xyz="0 0 -1"/>
     <limit lower="${-pi2*4}" upper="${pi2*4}" effort="10" velocity="6"/>
@@ -47,5 +146,6 @@
     <parent link="cgo3_vertical_arm_link"/>
     <child link="cgo3_horizontal_arm_link"/>
-    <origin xyz="0 0 0" rpy="0 0 0"/>
+    <!-- each origin is this pivot minus the parent's -->
+    <origin xyz="${-yaw_px} 0 ${roll_pz}" rpy="0 0 0"/>
     <axis xyz="-1 0 0"/>
     <limit lower="${-pi2}" upper="${pi2}" effort="10" velocity="6"/>
@@ -54,5 +154,5 @@
     <parent link="cgo3_horizontal_arm_link"/>
     <child link="camera_link"/>
-    <origin xyz="0 0 0" rpy="0 0 0"/>
+    <origin xyz="${pitch_px} 0 ${pitch_pz - roll_pz}" rpy="0 0 0"/>
     <axis xyz="0 1 0"/>
     <limit lower="${-pi2}" upper="${pi2}" effort="10" velocity="6"/>
@@ -67,10 +167,11 @@
         optical y = camera_link -z  = aircraft down
         optical z = camera_link -x  = aircraft forward
-    which is what image geometry expects.
+    which is what image geometry expects. The origin moves from the pitch
+    pivot to the sensor, which is where the image is actually taken.
   -->
   <joint name="camera_optical_joint" type="fixed">
     <parent link="camera_link"/>
     <child link="camera_optical_frame"/>
-    <origin xyz="0 0 0" rpy="${-pi2} 0 ${pi2}"/>
+    <origin xyz="${lens_px - pitch_px} 0 0" rpy="${-pi2} 0 ${pi2}"/>
   </joint>
 </robot>
